Commit message: versie met bewegende robot

File: src/my_xarm_lite6/my_lite6_description/urdf/robotopstelling.urdf.xacro (robot description, xacro)
@@ -2,5 +2,5 @@
 <robot xmlns:xacro="http://wiki.ros.org/xacro">
   <xacro:macro name="robotopstelling" params="">
-    <xacro:property name="mesh_file" value="package://my_lite6_description/meshes/RobotOpstelling2.STL"/>
+    <xacro:property name="mesh_file" value="package://my_lite6_description/meshes/RobotOpstelling4.STL"/>
     <xacro:property name="mesh_scale" value="1 1 1"/>
     <link name="robotopstelling_link">
