Commit message: Programma uitsorteren kwast 1-7

File: src/my_xarm_lite6/my_lite6_description/urdf/lite6_robot.urdf.xacro (robot description, xacro)
@@ -147,4 +147,30 @@
   <xacro:include filename="$(find xarm_description)/urdf/gripper/lite_gripper.urdf.xacro" />
   <xacro:uflite_gripper_urdf prefix="$(arg prefix)" attach_to='link_eef' />
+<!-- Gripper Link
+<link name="gripper_link">
+  <visual>
+    <origin xyz="-0.1026 -0.0806 -0.04175" rpy="0 0 0"/>
+    <geometry>
+      <mesh filename="package://my_lite6_description/meshes/gripper.stl" scale="0.001 0.001 0.001"/>
+    </geometry>
+    <material name="white"/>
+  </visual>
+  <collision>
+  <origin xyz="-0.1026 -0.0846 -0.04175" rpy="0 0 0"/>
+  <geometry>
+    <mesh filename="package://my_lite6_description/meshes/gripper.stl" scale="0.001 0.001 0.001"/>
+  </geometry>
+</collision>
+  <inertial>
+    <mass value="0.1"/>
+    <inertia ixx="0.001" iyy="0.001" izz="0.001" ixy="0" ixz="0" iyz="0"/>
+  </inertial>
+</link>
+<joint name="gripper_joint" type="fixed">
+  <parent link="link_eef"/>
+  <child link="gripper_link"/>
+  <origin xyz="0 0 0" rpy="-1.5708 0 0"/>
+</joint>
+-->
 <!-- Include jouw eigen robotopstelling -->
 <xacro:include filename="$(find my_lite6_description)/urdf/robotopstelling.urdf.xacro" />

File: src/my_xarm_lite6/my_lite6_description/urdf/robotopstelling.urdf.xacro (robot description, xacro)
@@ -2,5 +2,5 @@
 <robot xmlns:xacro="http://wiki.ros.org/xacro">
   <xacro:macro name="robotopstelling" params="">
-    <xacro:property name="mesh_file" value="package://my_lite6_description/meshes/RobotOpstelling4.STL"/>
+    <xacro:property name="mesh_file" value="package://my_lite6_description/meshes/RobotOpstelling10.STL"/>
     <xacro:property name="mesh_scale" value="1 1 1"/>
     <link name="robotopstelling_link">

File: src/xarm_ros/xarm_description/urdf/gripper/lite_gripper.urdf.xacro (robot description, xacro)
@@ -19,11 +19,11 @@
       <xacro:common_link_visual
         mesh_filename="gripper/lite/visual/gripper_lite"
-        origin_xyz="0.12 0.096 -0.015"
-        origin_rpy="0 0 3.14"
+        origin_xyz="-0.12 -0.038 0"
+        origin_rpy="0 0 0"
         material_name="${prefix}White" />
       <xacro:common_link_collision
         mesh_filename="gripper/lite/collision/gripper_lite"
-        origin_xyz="0.12 0.096 -0.015"
-        origin_rpy="0 0 3.14" />
+        origin_xyz="-0.12 -0.038 0"
+        origin_rpy="0 0 0" />
     </link>
     <link name="${prefix}link_tcp" />

Commit message: Robot controller V2

File: src/my_xarm_lite6/my_lite6_description/urdf/lite6_robot.urdf.xacro (robot description, xacro)
@@ -147,32 +147,9 @@
   <xacro:include filename="$(find xarm_description)/urdf/gripper/lite_gripper.urdf.xacro" />
   <xacro:uflite_gripper_urdf prefix="$(arg prefix)" attach_to='link_eef' />
-<!-- Gripper Link
-<link name="gripper_link">
-  <visual>
-    <origin xyz="-0.1026 -0.0806 -0.04175" rpy="0 0 0"/>
-    <geometry>
-      <mesh filename="package://my_lite6_description/meshes/gripper.stl" scale="0.001 0.001 0.001"/>
-    </geometry>
-    <material name="white"/>
-  </visual>
-  <collision>
-  <origin xyz="-0.1026 -0.0846 -0.04175" rpy="0 0 0"/>
-  <geometry>
-    <mesh filename="package://my_lite6_description/meshes/gripper.stl" scale="0.001 0.001 0.001"/>
-  </geometry>
-</collision>
-  <inertial>
-    <mass value="0.1"/>
-    <inertia ixx="0.001" iyy="0.001" izz="0.001" ixy="0" ixz="0" iyz="0"/>
-  </inertial>
-</link>
-<joint name="gripper_joint" type="fixed">
-  <parent link="link_eef"/>
-  <child link="gripper_link"/>
-  <origin xyz="0 0 0" rpy="-1.5708 0 0"/>
-</joint>
--->
 <!-- Include jouw eigen robotopstelling -->
 <xacro:include filename="$(find my_lite6_description)/urdf/robotopstelling.urdf.xacro" />
 <xacro:robotopstelling/>
+<!-- camera -->
+<xacro:include filename="$(find my_lite6_description)/urdf/camera.urdf.xacro" />
+<xacro:camera/>
 </robot>

File: src/my_xarm_lite6/my_lite6_description/urdf/robotopstelling.urdf.xacro (robot description, xacro)
@@ -2,5 +2,5 @@
 <robot xmlns:xacro="http://wiki.ros.org/xacro">
   <xacro:macro name="robotopstelling" params="">
-    <xacro:property name="mesh_file" value="package://my_lite6_description/meshes/RobotOpstelling10.STL"/>
+    <xacro:property name="mesh_file" value="package://my_lite6_description/meshes/RobotOpstelling11.STL"/>
     <xacro:property name="mesh_scale" value="1 1 1"/>
     <link name="robotopstelling_link">
