Commit message: my_depthai mapje 2

File: src/my_xarm_lite6/my_lite6_description/urdf/camera.urdf.xacro (robot description, xacro)
@@ -28,5 +28,5 @@
       <parent link="world"/>
       <child link="camera_link"/>
-      <origin xyz="0.1475 0.0775 0.8475" rpy="3.14 0 -1.57"/>
+      <origin xyz="0.1475 0.0205 0.8475" rpy="3.14 0 -1.57"/>
     </joint>
   </xacro:macro>
